Commit message: initial push

File: mtu32_description/urdf/robot_description.urdf.xacro (robot description, xacro)
@@ -10,7 +10,7 @@
   </visual>
   <collision>
-    <material name="clearpath_black"/>
+    <origin xyz="0 0.24 0.24" rpy="0 0 0"/>
     <geometry>
-      <mesh filename="package://mtu32_description/meshes/sensor_arch.stl"/>
+      <box size="0.17 0.05 0.2"/>
     </geometry>
   </collision>
@@ -22,3 +22,24 @@
   <origin xyz="0 0 0" rpy="0 0 0"/>
 </joint>
+<!-- Add Duro Base and E-Stop Button Link -->
+<link name="estop_link">
+  <visual>
+    <material name="clearpath_yellow"/>
+    <geometry>
+      <mesh filename="package://mtu32_description/meshes/duro_estop.stl"/>
+    </geometry>
+ </visual>
+  <collision>
+    <origin xyz="-0.28 0 0.37" rpy="0 0 0"/>
+    <geometry>
+      <box size="0.12 0.59 0.24"/>
+    </geometry>
+  </collision>
+</link>
+<!-- Add Mount Plates Joint -->
+<joint name="estop_joint" type="fixed">
+  <child link="estop_link"/>
+  <parent link="base_link"/>
+  <origin xyz="0 0 0" rpy="0 0 0"/>
+</joint>
 </robot>

Commit message: updates to meshes and URDF

File: mtu32_description/urdf/robot_description.urdf.xacro (robot description, xacro)
@@ -6,5 +6,5 @@
     <material name="clearpath_black"/>
     <geometry>
-      <mesh filename="package://mtu32_description/meshes/sensor_arch.stl"/>
+      <mesh filename="package://mtu32_description/meshes/sensor_arch.STL"/>
     </geometry>
   </visual>
@@ -27,5 +27,5 @@
     <material name="clearpath_yellow"/>
     <geometry>
-      <mesh filename="package://mtu32_description/meshes/duro_estop.stl"/>
+      <mesh filename="package://mtu32_description/meshes/duro_estop.STL"/>
     </geometry>
  </visual>
@@ -37,5 +37,5 @@
   </collision>
 </link>
-<!-- Add Mount Plates Joint -->
+<!-- Add Duro Base and E-Stop Button Joint -->
 <joint name="estop_joint" type="fixed">
   <child link="estop_link"/>
@@ -43,3 +43,18 @@
   <origin xyz="0 0 0" rpy="0 0 0"/>
 </joint>
+<!-- Add Duro Base and E-Stop Button Link -->
+<link name="button_link">
+  <visual>
+    <material name="clearpath_red"/>
+    <geometry>
+      <mesh filename="package://mtu32_description/meshes/button.STL"/>
+    </geometry>
+ </visual>
+</link>
+<!-- Add Duro Base and E-Stop Button Joint -->
+<joint name="button_joint" type="fixed">
+  <child link="button_link"/>
+  <parent link="base_link"/>
+  <origin xyz="0 0 0" rpy="0 0 0"/>
+</joint>
 </robot>

Commit message: udpates to meshes and URDF

File: mtu32_description/urdf/robot_description.urdf.xacro (robot description, xacro)
@@ -10,7 +10,7 @@
   </visual>
   <collision>
-    <origin xyz="0 0.24 0.24" rpy="0 0 0"/>
+    <origin xyz="0 0.235 0.17" rpy="0 0 0"/>
     <geometry>
-      <box size="0.17 0.05 0.2"/>
+      <box size="0.17 0.05 0.145"/> #antenna box
     </geometry>
   </collision>
@@ -31,7 +31,7 @@
  </visual>
   <collision>
-    <origin xyz="-0.28 0 0.37" rpy="0 0 0"/>
+    <origin xyz="0.32 0 0.4" rpy="0 0 0"/>
     <geometry>
-      <box size="0.12 0.59 0.24"/>
+      <box size="0.12 0.59 0.3"/> #main sensor arch box
     </geometry>
   </collision>
@@ -51,4 +51,10 @@
     </geometry>
  </visual>
+  <collision>
+    <origin xyz="0.2 0 0.31" rpy="0 0 0"/>
+    <geometry>
+      <box size="0.12 0.42 0.12"/> #cable protection box
+    </geometry>
+  </collision>
 </link>
 <!-- Add Duro Base and E-Stop Button Joint -->
@@ -58,3 +64,18 @@
   <origin xyz="0 0 0" rpy="0 0 0"/>
 </joint>
+<!-- Add Collision for Arm Ethernet Cable Link -->
+<link name="eth_link">
+  <collision>
+    <origin xyz="-0.2 -0.1 0.29226" rpy="0 0 0"/>
+    <geometry>
+      <box size="0.1 0.1 0.1"/> #am ethernet connection protection box
+    </geometry>
+  </collision>
+</link>
+<!-- Add Arm Ethernet Cable Joint -->
+<joint name="eth_joint" type="fixed">
+  <child link="eth_link"/>
+  <parent link="base_link"/>
+  <origin xyz="0 0 0" rpy="0 0 0"/>
+</joint>
 </robot>
