Commit message: top plate added

File: mtu32_description/urdf/robot_description_j100.urdf.xacro (robot description, xacro)
@@ -1,8 +1,30 @@
 <?xml version="1.0"?>
 <robot xmlns:xacro="http://ros.org/wiki/xacro">
+<!-- Add Mount Plates Link -->
+<link name="top_mount_link">
+  <visual>
+    <material name="clearpath_black"/>
+    <geometry>
+      <mesh filename="package://mtu32_description/meshes/top_mount_link.stl"/>
+    </geometry>
+  </visual>
+  <!-- <collision>
+    <origin xyz="0 0.235 0.17" rpy="0 0 0"/>
+    <geometry>
+      <box size="0.17 0.05 0.145"/> #antenna box
+    </geometry>
+  </collision> -->
+</link>
+<!-- Add Mount Plates Joint -->
+<joint name="top_mount_joint" type="fixed">
+  <child link="top_mount_link"/>
+  <parent link="default_mount"/>
+  <origin xyz="0 0 0.02" rpy="0 0 0"/>
+</joint>
+<!-- camera_1 -->
 <xacro:include filename="$(find mtu32_description)/urdf/intel_realsense.urdf.xacro"/>
 <xacro:intel_realsense name="camera_1" parent_link="arm_0_end_effector_link" update_rate="30" image_height="480" image_width="640" model="d405">
     <origin xyz="0.045 0.0 0.0" rpy="0.0 0.0 0.0"/>
     <!-- <origin xyz="0.055 -0.02 0.02" rpy="-1.5708 0.0 0.0"/> -->
-  </xacro:intel_realsense>
+</xacro:intel_realsense>
 </robot>

Commit message: fix

File: mtu32_description/urdf/robot_description_j100.urdf.xacro (robot description, xacro)
@@ -6,5 +6,5 @@
     <material name="clearpath_black"/>
     <geometry>
-      <mesh filename="package://mtu32_description/meshes/top_mount_link.stl"/>
+      <mesh filename="package://mtu32_description/meshes/jackal_top_assy_v1.stl"/>
     </geometry>
   </visual>

Commit message: collision added

File: mtu32_description/urdf/robot_description_j100.urdf.xacro (robot description, xacro)
@@ -4,4 +4,5 @@
 <link name="top_mount_link">
   <visual>
+    <origin xyz="0.067 0.024 0.124" rpy="1.5708 0.0 1.5708"/>
     <material name="clearpath_black"/>
     <geometry>
@@ -9,4 +10,10 @@
     </geometry>
   </visual>
+  <collision>
+    <origin xyz="0.067 0.024 0.124" rpy="1.5708 0.0 1.5708"/>
+    <geometry>
+      <mesh filename="package://mtu32_description/meshes/jackal_top_assy_v1.stl"/>
+    </geometry>
+  </collision>
   <!-- <collision>
     <origin xyz="0 0.235 0.17" rpy="0 0 0"/>
@@ -20,5 +27,6 @@
   <child link="top_mount_link"/>
   <parent link="default_mount"/>
-  <origin xyz="0 0 0.02" rpy="0 0 0"/>
+  <origin xyz="0.0 0.0 0.0" rpy="0.0 0.0 0.0"/>
+  <!-- <origin xyz="0.067 0.024 0.124" rpy="1.5708 0.0 1.5708"/> -->
 </joint>
 <!-- camera_1 -->

Commit message: top plate urdf

File: mtu32_description/urdf/robot_description_j100.urdf.xacro (robot description, xacro)
@@ -4,5 +4,5 @@
 <link name="top_mount_link">
   <visual>
-    <origin xyz="0.067 0.024 0.124" rpy="1.5708 0.0 1.5708"/>
+    <origin xyz="0.067 0.025 0.095" rpy="1.5708 0.0 1.5708"/>
     <material name="clearpath_black"/>
     <geometry>
@@ -11,15 +11,9 @@
   </visual>
   <collision>
-    <origin xyz="0.067 0.024 0.124" rpy="1.5708 0.0 1.5708"/>
+    <origin xyz="0.067 0.025 0.095" rpy="1.5708 0.0 1.5708"/>
     <geometry>
       <mesh filename="package://mtu32_description/meshes/jackal_top_assy_v1.stl"/>
     </geometry>
   </collision>
-  <!-- <collision>
-    <origin xyz="0 0.235 0.17" rpy="0 0 0"/>
-    <geometry>
-      <box size="0.17 0.05 0.145"/> #antenna box
-    </geometry>
-  </collision> -->
 </link>
 <!-- Add Mount Plates Joint -->
@@ -27,5 +21,5 @@
   <child link="top_mount_link"/>
   <parent link="default_mount"/>
-  <origin xyz="0.0 0.0 0.0" rpy="0.0 0.0 0.0"/>
+  <origin xyz="0.0 0.0 0.028" rpy="0.0 0.0 0.0"/>
   <!-- <origin xyz="0.067 0.024 0.124" rpy="1.5708 0.0 1.5708"/> -->
 </joint>

Commit message: new top mesh

File: mtu32_description/urdf/robot_description_j100.urdf.xacro (robot description, xacro)
@@ -7,5 +7,5 @@
     <material name="clearpath_black"/>
     <geometry>
-      <mesh filename="package://mtu32_description/meshes/jackal_top_assy_v1.stl"/>
+      <mesh filename="package://mtu32_description/meshes/top_assy_duro_ant.stl"/>
     </geometry>
   </visual>
@@ -13,5 +13,5 @@
     <origin xyz="0.067 0.025 0.095" rpy="1.5708 0.0 1.5708"/>
     <geometry>
-      <mesh filename="package://mtu32_description/meshes/jackal_top_assy_v1.stl"/>
+      <mesh filename="package://mtu32_description/meshes/top_assy_duro_ant.stl"/>
     </geometry>
   </collision>

Commit message: jackal new top plate mesh adjusted

File: mtu32_description/urdf/robot_description_j100.urdf.xacro (robot description, xacro)
@@ -4,14 +4,14 @@
 <link name="top_mount_link">
   <visual>
-    <origin xyz="0.067 0.025 0.095" rpy="1.5708 0.0 1.5708"/>
+    <origin xyz="0.0 0.0 0.0" rpy="0.0 0.0 3.14159"/>
     <material name="clearpath_black"/>
     <geometry>
-      <mesh filename="package://mtu32_description/meshes/top_assy_duro_ant.stl"/>
+      <mesh filename="package://mtu32_description/meshes/top_assy_duro_ant.stl"  scale="0.001 0.001 0.001"/>
     </geometry>
   </visual>
   <collision>
-    <origin xyz="0.067 0.025 0.095" rpy="1.5708 0.0 1.5708"/>
+    <origin xyz="0.0 0.0 0.0" rpy="0.0 0.0 3.14159"/>
     <geometry>
-      <mesh filename="package://mtu32_description/meshes/top_assy_duro_ant.stl"/>
+      <mesh filename="package://mtu32_description/meshes/top_assy_duro_ant.stl"  scale="0.001 0.001 0.001"/>
     </geometry>
   </collision>

Commit message: new top plate rev 1

File: mtu32_description/urdf/robot_description_j100.urdf.xacro (robot description, xacro)
@@ -7,5 +7,5 @@
     <material name="clearpath_black"/>
     <geometry>
-      <mesh filename="package://mtu32_description/meshes/top_assy_duro_ant.stl"  scale="0.001 0.001 0.001"/>
+      <mesh filename="package://mtu32_description/meshes/top_assy_rev1.dae"  scale="0.001 0.001 0.001"/>
     </geometry>
   </visual>
@@ -13,5 +13,5 @@
     <origin xyz="0.0 0.0 0.0" rpy="0.0 0.0 3.14159"/>
     <geometry>
-      <mesh filename="package://mtu32_description/meshes/top_assy_duro_ant.stl"  scale="0.001 0.001 0.001"/>
+      <mesh filename="package://mtu32_description/meshes/top_assy_rev1.dae"  scale="0.001 0.001 0.001"/>
     </geometry>
   </collision>
