Commit message: mapless nav settings

File: mtu32_description/urdf/robot_description_j100.urdf.xacro (robot description, xacro)
@@ -25,8 +25,8 @@
 </joint>
 <!-- camera_1 -->
-<xacro:include filename="$(find mtu32_description)/urdf/intel_realsense.urdf.xacro"/>
+<!-- <xacro:include filename="$(find mtu32_description)/urdf/intel_realsense.urdf.xacro"/>
 <xacro:intel_realsense name="camera_1" parent_link="arm_0_end_effector_link" update_rate="30" image_height="480" image_width="640" model="d405">
-    <origin xyz="0.045 0.0 0.0" rpy="0.0 0.0 0.0"/>
+    <origin xyz="0.045 0.0 0.0" rpy="0.0 0.0 0.0"/> -->
     <!-- <origin xyz="0.055 -0.02 0.02" rpy="-1.5708 0.0 0.0"/> -->
-</xacro:intel_realsense>
+<!-- </xacro:intel_realsense> -->
 </robot>

Commit message: outdoor ready

File: mtu32_description/urdf/robot_description_j100.urdf.xacro (robot description, xacro)
@@ -25,8 +25,8 @@
 </joint>
 <!-- camera_1 -->
-<!-- <xacro:include filename="$(find mtu32_description)/urdf/intel_realsense.urdf.xacro"/>
+<xacro:include filename="$(find mtu32_description)/urdf/intel_realsense.urdf.xacro"/>
 <xacro:intel_realsense name="camera_1" parent_link="arm_0_end_effector_link" update_rate="30" image_height="480" image_width="640" model="d405">
-    <origin xyz="0.045 0.0 0.0" rpy="0.0 0.0 0.0"/> -->
+    <origin xyz="0.045 0.0 0.0" rpy="0.0 0.0 0.0"/>
     <!-- <origin xyz="0.055 -0.02 0.02" rpy="-1.5708 0.0 0.0"/> -->
-<!-- </xacro:intel_realsense> -->
+</xacro:intel_realsense>
 </robot>

Commit message: gps IP change

File: mtu32_description/urdf/robot_description_j100.urdf.xacro (robot description, xacro)
@@ -27,5 +27,6 @@
 <xacro:include filename="$(find mtu32_description)/urdf/intel_realsense.urdf.xacro"/>
 <xacro:intel_realsense name="camera_1" parent_link="arm_0_end_effector_link" update_rate="30" image_height="480" image_width="640" model="d405">
-    <origin xyz="0.045 0.0 0.0" rpy="0.0 0.0 0.0"/>
+    <origin xyz="-0.036 0.0 0.059" rpy="1.5708 -1.5708 -1.5708"/>
+    <!-- <origin xyz="0.045 0.0 0.0" rpy="0.0 0.0 0.0"/> -->
     <!-- <origin xyz="0.055 -0.02 0.02" rpy="-1.5708 0.0 0.0"/> -->
 </xacro:intel_realsense>
