Commit message: Snapshot for multirobot_sim: sim_robot_upstart launch, MoveIt/servo configs, working-copy edits from j100_0921
Branched from j100_0921 so the real robot's branch stays untouched. Includes
sim_robot_upstart.launch.py (Isaac Sim bringup), moveit/servo/pcl launch and
config files, and the robot's uncommitted working-copy edits copied from
robot_data/j100_0921.

Co-Authored-By: Claude Opus 5.5 <noreply@anthropic.com>

File: mtu32_description/urdf/robot_description_j100.urdf.xacro (robot description, xacro)
@@ -27,7 +27,6 @@
 <xacro:include filename="$(find mtu32_description)/urdf/intel_realsense.urdf.xacro"/>
 <xacro:intel_realsense name="camera_1" parent_link="arm_0_end_effector_link" update_rate="30" image_height="480" image_width="640" model="d405">
-    <origin xyz="-0.036 0.0 0.059" rpy="1.5708 -1.5708 -1.5708"/>
-    <!-- <origin xyz="0.045 0.0 0.0" rpy="0.0 0.0 0.0"/> -->
-    <!-- <origin xyz="0.055 -0.02 0.02" rpy="-1.5708 0.0 0.0"/> -->
+    <!-- <origin xyz="-0.036 0.0 -0.059" rpy="1.5708 -1.5708 -1.5708"/> -->
+    <origin xyz="-0.048 0.0 -0.003" rpy="1.5708 -1.5708 -1.5708"/>
 </xacro:intel_realsense>
 </robot>

Commit message: j100 cutter EE: visual + MoveIt collision envelope, finger pairs disabled
mtu32_description: ee_cutter_link on arm_0_gripper_gripper_base_link (the
cutter + gripper EE that replaces the 2F Lite fingers): its static parts as
a mesh and its envelope as 8 boxes from the STEP for MoveIt; the 7 moving
bodies (crossbar, pusher, link_1, link_2, finger tip, blade, spur gear) on
fixed ee_cutter_<body>_joint at their CAD pivots (the sim animates them in
its published robot_description; a real robot publishes no state for them).
Meshes from multirobot_sim's sim/scripts/make_ee_cutter_urdf_mesh.py.

moveit.launch.py: with ee_cutter_link in the URDF, disable its collisions
with every arm_0_gripper_*_finger_* link: the generated SRDF missed
left_finger_dist, MoveIt saw the closed gripper in collision and Servo
stopped every cut.

Co-Authored-By: Claude Opus 5.5 <noreply@anthropic.com>

File: mtu32_description/urdf/robot_description_j100.urdf.xacro (robot description, xacro)
@@ -30,3 +30,110 @@
     <origin xyz="-0.048 0.0 -0.003" rpy="1.5708 -1.5708 -1.5708"/>
 </xacro:intel_realsense>
+<!-- Cutter + gripper end effector (replaces the 2F Lite's fingers; their links stay, MoveIt and the arm driver
+     command its finger joint). Visual: the EE's static parts (sim/scripts/make_ee_cutter_urdf_mesh.py; the moving ones
+     follow below). Collision: its envelope as boxes from the STEP (cutter_and_gripper_and_camera_bracket
+     .stp, CAD frame: x -> y, y -> z, z -> x, +2.2 mm in z) for MoveIt; finger_sweep covers the finger tip's whole
+     travel, the jaw opening is filled (MoveIt sees no stems). -->
+<link name="ee_cutter_link">
+  <visual>
+    <origin xyz="0 0 0" rpy="0 0 0"/>
+    <geometry><mesh filename="package://mtu32_description/meshes/ee_cutter.obj"/></geometry>
+  </visual>
+  <collision name="housing">
+    <origin xyz="0.0340 -0.0040 0.0692" rpy="0 0 0"/>
+    <geometry><box size="0.0360 0.1460 0.1340"/></geometry>
+  </collision>
+  <collision name="housing_rear">
+    <origin xyz="0.0410 -0.0040 -0.0118" rpy="0 0 0"/>
+    <geometry><box size="0.0160 0.1460 0.0280"/></geometry>
+  </collision>
+  <collision name="dynamixel">
+    <origin xyz="0.0635 -0.0050 0.0687" rpy="0 0 0"/>
+    <geometry><box size="0.0230 0.0480 0.0550"/></geometry>
+  </collision>
+  <collision name="blades">
+    <origin xyz="0.0350 0.0025 0.1547" rpy="0 0 0"/>
+    <geometry><box size="0.0140 0.1250 0.0370"/></geometry>
+  </collision>
+  <collision name="jaw_linkage">
+    <origin xyz="0.0000 -0.0230 0.0892" rpy="0 0 0"/>
+    <geometry><box size="0.0260 0.1220 0.1340"/></geometry>
+  </collision>
+  <collision name="finger_sweep">
+    <origin xyz="0.0070 -0.0185 0.1892" rpy="0 0 0"/>
+    <geometry><box size="0.0300 0.0970 0.0660"/></geometry>
+  </collision>
+  <collision name="fixtures">
+    <origin xyz="0.0000 0.0000 0.0202" rpy="0 0 0"/>
+    <geometry><box size="0.0720 0.0800 0.0360"/></geometry>
+  </collision>
+  <collision name="d405_bracket">
+    <origin xyz="-0.0470 0.0000 0.0102" rpy="0 0 0"/>
+    <geometry><box size="0.0220 0.0490 0.0500"/></geometry>
+  </collision>
+</link>
+<joint name="ee_cutter_joint" type="fixed">
+  <parent link="arm_0_gripper_gripper_base_link"/>
+  <child link="ee_cutter_link"/>
+  <origin xyz="0 0 0" rpy="0 0 0"/>
+</joint>
+<!-- The EE's moving bodies (sim/scripts/ee_cutter.py BODIES), each at its CAD pivot: fixed here (a real robot
+     publishes no state for them, and MoveIt would wait for one); the sim's robot_state makes them prismatic /
+     revolute (axis z / x) in the published robot_description, and they follow the sim's platform/joint_states. -->
+<link name="ee_cutter_slide_link">
+  <visual><geometry><mesh filename="package://mtu32_description/meshes/ee_cutter_slide.obj"/></geometry></visual>
+</link>
+<joint name="ee_cutter_slide_joint" type="fixed">
+  <parent link="ee_cutter_link"/>
+  <child link="ee_cutter_slide_link"/>
+  <origin xyz="0.00000 0.00000 0.00220" rpy="0 0 0"/>
+</joint>
+<link name="ee_cutter_pusher_link">
+  <visual><geometry><mesh filename="package://mtu32_description/meshes/ee_cutter_pusher.obj"/></geometry></visual>
+</link>
+<joint name="ee_cutter_pusher_joint" type="fixed">
+  <parent link="ee_cutter_slide_link"/>
+  <child link="ee_cutter_pusher_link"/>
+  <origin xyz="0.00000 -0.05103 0.05555" rpy="0 0 0"/>
+</joint>
+<link name="ee_cutter_link_1_link">
+  <visual><geometry><mesh filename="package://mtu32_description/meshes/ee_cutter_link_1.obj"/></geometry></visual>
+</link>
+<joint name="ee_cutter_link_1_joint" type="fixed">
+  <parent link="ee_cutter_link"/>
+  <child link="ee_cutter_link_1_link"/>
+  <origin xyz="0.00000 -0.04443 0.11000" rpy="0 0 0"/>
+</joint>
+<link name="ee_cutter_link_2_link">
+  <visual><geometry><mesh filename="package://mtu32_description/meshes/ee_cutter_link_2.obj"/></geometry></visual>
+</link>
+<joint name="ee_cutter_link_2_joint" type="fixed">
+  <parent link="ee_cutter_link_1_link"/>
+  <child link="ee_cutter_link_2_link"/>
+  <origin xyz="0.00000 -0.03300 -0.02259" rpy="0 0 0"/>
+</joint>
+<link name="ee_cutter_finger_link">
+  <visual><geometry><mesh filename="package://mtu32_description/meshes/ee_cutter_finger.obj"/></geometry></visual>
+</link>
+<joint name="ee_cutter_finger_joint" type="fixed">
+  <parent link="ee_cutter_link"/>
+  <child link="ee_cutter_finger_link"/>
+  <origin xyz="0.00000 -0.04448 0.15000" rpy="0 0 0"/>
+</joint>
+<link name="ee_cutter_blade_link">
+  <visual><geometry><mesh filename="package://mtu32_description/meshes/ee_cutter_blade.obj"/></geometry></visual>
+</link>
+<joint name="ee_cutter_blade_joint" type="fixed">
+  <parent link="ee_cutter_link"/>
+  <child link="ee_cutter_blade_link"/>
+  <origin xyz="0.00000 0.00593 0.10824" rpy="0 0 0"/>
+</joint>
+<link name="ee_cutter_spur_link">
+  <visual><geometry><mesh filename="package://mtu32_description/meshes/ee_cutter_spur.obj"/></geometry></visual>
+</link>
+<joint name="ee_cutter_spur_joint" type="fixed">
+  <parent link="ee_cutter_link"/>
+  <child link="ee_cutter_spur_link"/>
+  <origin xyz="0.00000 0.00085 0.05800" rpy="0 0 0"/>
+</joint>
 </robot>
